File: hotdoggu_smolSlimeVR.kicad_pcb (KiCad board)
At the start: 2 copper layers, 35 x 40 mm, 47 parts, among them J1 TYPE-C-31-M-12, J2 BATT, SW1 SW_SPDT, SW2 TS-1088-AR02016, SW3 TS-1088-AR02016, U1 ESP32-C3-MINI-1, U2 TPS63900, U3 TP4056-42-ESOP8, U4 DW01A, U5 FS8205, U6 LSM6DSV16X

Commit message: Hotdoggu_smolSlimeVR V2
Parts:
- removed C3: 100nF, Capacitor_SMD:C_0402_1005Metric
- removed C4: 10uF, Capacitor_SMD:C_0805_2012Metric
- removed D4, D5, D6: 1N5819WS, Diode_SMD:D_SOD-323
- removed L1: 2.2uH, Inductor_SMD:L_Murata_DFE201610P
- removed LED4: LED,0603,White, LED_SMD:LED_0603_1608Metric
- removed R1: 36.5k, 1%, Resistor_SMD:R_0402_1005Metric
- removed R10, R9: 33R, 1%, Resistor_SMD:R_0402_1005Metric
- removed R4, R8: 1k, Resistor_SMD:R_0402_1005Metric
- removed R6: 1.2k, Resistor_SMD:R_0402_1005Metric
- removed R7: 100, Resistor_SMD:R_0402_1005Metric
- removed U5: FS8205, Package_TO_SOT_SMD:SOT-23-6
- removed U6: LSM6DSV16X, Package_LGA:LGA-14_3x2.5mm_P0.5mm_LayoutBorder3x4y
- added C8: 100nF, Capacitor_SMD:C_0603_1608Metric, F.Cu at (173.0, 68.0)
- added R19: 2k, Resistor_SMD:R_0603_1608Metric, F.Cu at (168.0, 94.0)
- added REF**: IMU_XYZ, hotdoggu_smolSlimeVR:IMU_XYZ, F.Cu at (160.8, 87.4)
- C1, C5, C6, C7: footprint Capacitor_SMD:C_0402_1005Metric -> Capacitor_SMD:C_0603_1608Metric
- C2: value 22uF -> 10uF; footprint Capacitor_SMD:C_0402_1005Metric -> Capacitor_SMD:C_0603_1608Metric
- H2: footprint MountingHole:MountingHole_2.2mm_M2_DIN965 -> MountingHole:MountingHole_2.2mm_M2_DIN965_Pad_TopBottom
- J1: footprint hotdoggu_smolSlimeVR:TYPE-C-31-M-12 -> Connector_USB:USB_C_Receptacle_GCT_USB4105-xx-A_16P_TopMnt_Horizontal
- J2: value BATT -> 53261-0271
- LED2: value LED,0603,Yellow -> 0603,Yellow
- LED3: value LED,0603,Green -> 0603,White
- R11, R12: value 5.5k, 1% -> 1k; footprint Resistor_SMD:R_0402_1005Metric -> Resistor_SMD:R_0603_1608Metric
- R13, R14, R17, R18, R2, R3: footprint Resistor_SMD:R_0402_1005Metric -> Resistor_SMD:R_0603_1608Metric
- R15, R16: value 100 -> 1k, 1%; footprint Resistor_SMD:R_0402_1005Metric -> Resistor_SMD:R_0603_1608Metric
- R5: value 1k -> 5.1k; footprint Resistor_SMD:R_0402_1005Metric -> Resistor_SMD:R_0603_1608Metric
- SW1: value SW_SPDT -> JS202011CQN; footprint hotdoggu_smolSlimeVR:MSL_1C2P -> Button_Switch_THT:SW_CK_JS202011CQN_DPDT_Straight
- U2: value TPS63900 -> LSM6DSV16X; footprint Package_SON:WSON-10-1EP_2.5x2.5mm_P0.5mm_EP1.2x2mm_ThermalVias -> Package_LGA:LGA-14_3x2.5mm_P0.5mm_LayoutBorder3x4y
- U3: value TP4056-42-ESOP8 -> MCP73831-2-OT; footprint Package_SO:SOIC-8-1EP_3.9x4.9mm_P1.27mm_EP2.41x3.3mm_ThermalVias -> Package_TO_SOT_SMD:SOT-23-5
- U4: value DW01A -> LP5907MFX-3.3; footprint Package_TO_SOT_SMD:SOT-23-6 -> Package_TO_SOT_SMD:SOT-23-5
- moved R13 19.9 mm to (155.0, 85.2), turned to -90 degrees
- moved R14 19.5 mm to (156.5, 85.2), turned to -90 degrees
- moved SW3 15.8 mm to (179.0, 68.8), turned to 180 degrees
- moved U2 13.8 mm to (166.0, 86.5), turned to 0 degrees
- moved R2 13.3 mm to (172.0, 84.7)
- moved J1 12.7 mm to (179.4, 83.0)
- moved R3 12.3 mm to (172.0, 80.7)
- moved SW2 12.1 mm to (179.0, 73.2), turned to 180 degrees
- moved U3 9.64 mm to (172.0, 94.5), turned to 90 degrees
- moved C6 9.60 mm to (164.5, 90.0), turned to 180 degrees
- moved U4 9.15 mm to (157.4, 94.4), turned to 0 degrees
- moved R17 6.78 mm to (173.0, 69.5), turned to 180 degrees
- moved C7 6.48 mm to (172.9, 73.8), turned to 0 degrees
- moved R18 6.04 mm to (172.9, 72.2), turned to 180 degrees
- moved C5 5.99 mm to (170.2, 87.2), turned to -90 degrees
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Connections:
- C1 pad 1: Net-(D6-A) -> /VIN
- C6 pad 1: GND -> +3V3
- C6 pad 2: +3V3 -> GND
- H1 pad 1: (no net) -> GND
- H3 pad 1: (no net) -> GND
- J1 pad A6: Net-(J1-D+-PadA6) -> /USB_D+
- J1 pad A7: Net-(J1-D--PadA7) -> /USB_D-
- J1 pad B6: Net-(J1-D+-PadA6) -> /USB_D+
- J1 pad B7: Net-(J1-D--PadA7) -> /USB_D-
- J2 pad 1: Net-(D5-K) -> /VBAT
- J2 pad 2: Net-(D4-A) -> GND
- LED1 pad 1: GND -> Net-(LED1-K)
- LED1 pad 2: Net-(LED1-A) -> +3V3
- LED2 pad 2: Net-(LED2-A) -> /VUSB
- LED3 pad 2: Net-(LED3-A) -> /STAT
- R11 pad 1: Net-(LED1-A) -> Net-(LED1-K)
- R11 pad 2: +3V3 -> GND
- R12 pad 1: Net-(LED4-A) -> GND
- R12 pad 2: Net-(U1-GPIO10) -> Net-(LED3-K)
- R15 pad 2: /BAT+ -> /VBATSW
- R5 pad 1: Net-(LED3-A) -> /BATT_STAT
- R5 pad 2: /VUSB -> Net-(LED2-K)
- SW1 pad 2: /BAT+ -> /VBAT
- SW1 pad 3: Net-(D6-A) -> /VBATSW
- SW2 pad 2: /~{BOOT} -> /~{RESET}
- SW3 pad 2: /~{RESET} -> /~{BOOT}
- U1 pad 16: Net-(U1-GPIO10) -> /STAT
- U1 pad 26: /USB_D+ -> /USB_D-
- U1 pad 27: /USB_D- -> /USB_D+
- U2 pad 1: Net-(D6-A) -> unconnected-(U2-SDO/SA0-Pad1)
- U2 pad 10: Net-(D6-A) -> unconnected-(U2-OCS_Aux-Pad10)
- U2 pad 11: GND -> unconnected-(U2-SDO_Aux-Pad11)
- U2 pad 2: Net-(D6-A) -> +3V3
- U2 pad 3: Net-(U2-CFG1) -> +3V3
- U2 pad 4: GND -> unconnected-(U2-INT1-Pad4)
- U2 pad 5: GND -> +3V3
- U2 pad 6: +3V3 -> GND
- U2 pad 7: Net-(U2-LX2) -> GND
- U2 pad 8: GND -> +3V3
- U2 pad 9: Net-(U2-LX1) -> unconnected-(U2-INT2-Pad9)
- U3 pad 1: GND -> /BATT_STAT
- U3 pad 2: Net-(U3-PROG) -> GND
- U3 pad 3: GND -> /VBAT
- U3 pad 5: /BAT+ -> Net-(U3-PROG)
- U4 pad 1: Net-(U4-OD) -> /VIN
- U4 pad 2: Net-(U4-CS) -> GND
- U4 pad 3: Net-(U4-OC) -> /VIN
- U4 pad 5: Net-(U4-VCC) -> +3V3
Routing:
- net +3V3: track 20.9 -> 107.7 mm, vias 8 -> 5
- net /VBAT: track 0.00 -> 33.0 mm, vias 0 -> 1
- net Net-(U1-GPIO10): track 32.7 -> 0.00 mm, vias 2 -> 0
- net /STAT: track 0.00 -> 32.1 mm, vias 0 -> 2
- net /~{RESET}: track 4.60 -> 36.7 mm, vias 0 -> 2
- net /BAT+: track 29.8 -> 0.00 mm
- net /~{BOOT}: track 2.28 -> 30.5 mm, vias 0 -> 2
- net /VUSB: track 57.3 -> 34.8 mm, vias 5 -> 4
- net Net-(D6-A): track 17.6 -> 0.00 mm, vias 2 -> 0
- net /VIN: track 0.00 -> 17.5 mm
- net Net-(LED2-K): track 17.9 -> 1.50 mm, vias 2 -> 0
- net Net-(LED3-K): track 17.8 -> 1.49 mm, vias 2 -> 0
- net Net-(D4-A): track 13.2 -> 0.00 mm
- net /VBATSW: track 0.00 -> 10.8 mm
- net /SCL: track 23.2 -> 14.4 mm
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- added copper zone on B.Cu, net GND
- removed copper zone on B.Cu, net +3V3
Other:
- outline, holes or cut-outs redrawn
- board text added: "B"
- board text added: "CHG"
- board text added: "Hotdoggu_smolSlimeVR LSM6DSV16X V2"
- board text added: "PWR"
- board text added: "R"
- board text added: "STAT"
- board text removed: "BOOT"
- board text removed: "RST"
