File: hotdoggu_smolSlimeVR.kicad_sch (KiCad schematic)
At the start: 47 parts, among them J1 TYPE-C-31-M-12, J2 BATT, SW1 SW_SPDT, SW2 TS-1088-AR02016, SW3 TS-1088-AR02016, U1 ESP32-C3-MINI-1, U2 TPS63900, U3 TP4056-42-ESOP8, U4 DW01A, U5 FS8205, U6 LSM6DSV16X

Commit message: Hotdoggu_smolSlimeVR V2
Parts:
- removed C3: 100nF, Capacitor_SMD:C_0402_1005Metric, symbol Device:C_Small
- removed C4: 10uF, Capacitor_SMD:C_0805_2012Metric, symbol Device:C_Small
- removed D4, D5, D6: 1N5819WS, Diode_SMD:D_SOD-323, symbol Device:D_Small
- removed L1: 2.2uH, Inductor_SMD:L_Murata_DFE201610P, symbol Device:L_Small
- removed LED3: LED,0603,Green, LED_SMD:LED_0603_1608Metric, symbol Device:LED
- removed R1: 36.5k, 1%, Resistor_SMD:R_0402_1005Metric, symbol Device:R_Small
- removed R10, R9: 33R, 1%, Resistor_SMD:R_0402_1005Metric, symbol Device:R_Small
- removed R4, R8: 1k, Resistor_SMD:R_0402_1005Metric, symbol Device:R_Small
- removed R6: 1.2k, Resistor_SMD:R_0402_1005Metric, symbol Device:R_Small
- removed R7: 100, Resistor_SMD:R_0402_1005Metric, symbol Device:R_Small
- removed SW1: SW_SPDT, hotdoggu_smolSlimeVR:MSL_1C2P, symbol Switch:SW_SPDT
- removed SW2: TS-1088-AR02016, hotdoggu_smolSlimeVR:TS-1088-AR02016, symbol Switch:SW_Push
- removed U2: TPS63900, Package_SON:WSON-10-1EP_2.5x2.5mm_P0.5mm_EP1.2x2mm_ThermalVias, symbol Regulator_Switching:TPS63900
- removed U3: TP4056-42-ESOP8, Package_SO:SOIC-8-1EP_3.9x4.9mm_P1.27mm_EP2.41x3.3mm_ThermalVias, symbol Battery_Management:TP4056-42-ESOP8
- removed U4: DW01A, Package_TO_SOT_SMD:SOT-23-6, symbol Battery_Management:DW01A
- removed U5: FS8205, Package_TO_SOT_SMD:SOT-23-6, symbol hotdoggu_smolSlimeVR:FS8205
- removed U6: LSM6DSV16X, Package_LGA:LGA-14_3x2.5mm_P0.5mm_LayoutBorder3x4y, symbol hotdoggu_smolSlimeVR:LSM6DSV16X
- added C8: 100nF, Capacitor_SMD:C_0603_1608Metric, symbol Device:C_Small
- added R19: 2k, Resistor_SMD:R_0603_1608Metric, symbol Device:R_Small
- added SW1: JS202011CQN, Button_Switch_THT:SW_CK_JS202011CQN_DPDT_Straight, symbol Switch:SW_Slide_DPDT
- added SW3: TS-1088-AR02016, hotdoggu_smolSlimeVR:TS-1088-AR02016, symbol Switch:SW_Push
- added U2: LSM6DSV16X, Package_LGA:LGA-14_3x2.5mm_P0.5mm_LayoutBorder3x4y, symbol hotdoggu_smolSlimeVR:LSM6DSV16X
- added U3: MCP73831-2-OT, Package_TO_SOT_SMD:SOT-23-5, symbol hotdoggu_smolSlimeVR:MCP73831-2-OT
- added U4: LP5907MFX-3.3, Package_TO_SOT_SMD:SOT-23-5, symbol hotdoggu_smolSlimeVR:LP5907MFX-3.3
- C1, C5, C6, C7: footprint Capacitor_SMD:C_0402_1005Metric -> Capacitor_SMD:C_0603_1608Metric
- C2: value 22uF -> 10uF; footprint Capacitor_SMD:C_0402_1005Metric -> Capacitor_SMD:C_0603_1608Metric
- H1, H3: symbol Mechanical:MountingHole -> Mechanical:MountingHole_Pad
- H2: footprint MountingHole:MountingHole_2.2mm_M2_DIN965 -> MountingHole:MountingHole_2.2mm_M2_DIN965_Pad_TopBottom; symbol Mechanical:MountingHole -> Mechanical:MountingHole_Pad
- J1: footprint hotdoggu_smolSlimeVR:TYPE-C-31-M-12 -> Connector_USB:USB_C_Receptacle_GCT_USB4105-xx-A_16P_TopMnt_Horizontal
- J2: value BATT -> 53261-0271
- LED2: value LED,0603,Yellow -> 0603,Yellow
- LED3: renamed from LED4; value LED,0603,White -> 0603,White
- R11, R12: value 5.5k, 1% -> 1k; footprint Resistor_SMD:R_0402_1005Metric -> Resistor_SMD:R_0603_1608Metric
- R13, R14, R17, R18, R2, R3: footprint Resistor_SMD:R_0402_1005Metric -> Resistor_SMD:R_0603_1608Metric
- R15, R16: value 100 -> 1k, 1%; footprint Resistor_SMD:R_0402_1005Metric -> Resistor_SMD:R_0603_1608Metric
- R5: value 1k -> 5.1k; footprint Resistor_SMD:R_0402_1005Metric -> Resistor_SMD:R_0603_1608Metric
- renumbered SW3 to SW2
Connections:
- net +3V3: now also C6.1, LED1.2 (A), U2.2 (SDX), U2.3 (SCX), U2.5 (VDDIO), U2.8 (VDD), U4.5 (OUT); no longer C6.2, R11.2
- net GND: now also C6.2, H1.1, H2.1, H3.1, J2.2 (Pin_2), R11.2, R12.1, C8.1, R19.1, SW3.1, U2.6 (GND), U2.7 (GND), U3.2 (V_{SS}), U4.2 (GND); no longer C6.1, LED1.1 (K), LED3.1 (K)
- net SCL: now also U2.13 (SCL)
- net SDA: now also U2.14 (SDA)
- net USB_D+: now also J1.A6 (D+), J1.B6 (D+), U1.27 (GPIO19/USB_D+); no longer U1.26 (GPIO18/USB_D-)
- net USB_D-: now also J1.A7 (D-), J1.B7 (D-), U1.26 (GPIO18/USB_D-); no longer U1.27 (GPIO19/USB_D+)
- net VUSB: now also LED2.2 (A), U3.4 (V_{DD}); no longer R5.2
- net ~{BOOT}: now also C8.2, SW3.2
- net STAT: now reaches LED3.2 (A)
- net STAT: now also U1.16 (GPIO10); no longer R12.1
- net VIN: now reaches C1.1
- net VIN: now also SW1.4 (A), U4.1 (IN), U4.3 (EN)
- net BATT_STAT: now reaches R5.1
- net BATT_STAT: now also U3.1 (STAT)
- net VBAT: now reaches J2.1 (Pin_1)
- net VBAT: now also SW1.2 (B), SW1.5 (B), U3.3 (V_{BAT})
- net at R12.2: now also LED3.1 (K); no longer U1.16 (GPIO10)
- net at LED2.1 (K): now also R5.2
- net at R11.1: now also LED1.1 (K); no longer LED1.2 (A)
- net BAT+ renamed VBATSW
- net VBATSW: now also SW1.3 (C)
- new net: R19.2, U3.5 (PROG)
Other:
- note added: "BATTERY CHARGER"
- note added: "LDO Step-Down Regulator"
- note added: "LEDs"
- note removed: "BATT CHG"
- note removed: "BATT MANAGEMENT"
- note removed: "BATT PROTECTION"
- note removed: "Buck Boost/Step-Down Regulator"
- moved on the sheet: C1, C5, C6, J2, LED1, LED2, LED3, R11, R12, R5
